File: PCB/KiCAD/PhoZL-2.0.2.kicad_pcb (KiCad board)
At the start: 2 copper layers, 125.5 x 90.3 mm, 108 parts, among them J1 Conn_01x06_Female, J11 Conn_01x02, J14 Conn_01x06, J15 Conn_01x06, J2 Conn_01x02, J3 Conn_01x02, J4 Conn_01x01, J5 Rumble, J6 Conn_01x06, J8 USB_B_Micro, Q1 Q_NMOS_GSD, Q2 Q_PMOS_GDS, Q3 Q_NMOS_GSD, SW1 A, SW10 Dup, SW11 Dright, SW12 Ddown, SW2 B, SW3 X, SW4 Y, SW5 Start, SW6 L, SW7 R, SW8 Z, SW9 Dleft, U1 MCP3002, U10 DRV5055A2xDBZxQ1, U11 DRV5055A2xDBZxQ1, U2 Stickbox_Assembly_Main, U3 MCP3002, U4 DRV5055A2xDBZxQ1, U5 Stickbox_Assembly_CStick, U6 AMS1117-3.3, U7 W25Q128JVS, U8 RP2040, U9 DRV5055A2xDBZxQ1, Y1 Crystal_GND24

Commit message: altered the files on my fork to reflect the changes described in changes.txt
Parts:
- removed Gphobtvbigback (x2): LOGO, Library:phobtv_bold_big
- removed Gtvsmallfrontc: LOGO, Library:phobtv_bold_smol
- added SW8L: ZL, PhobGCC_2_0_0_footprints:Z_Switch_Edge_Omron, F.Cu at (60.8, 35.5)
- SW8: value Z -> ZR
Routing:
- net /GPIO15: track 15.0 -> 89.1 mm, vias 0 -> 1
- net GND: track 131.9 -> 138.4 mm, vias 49 -> 48
- net /Din: track 125.5 -> 124.9 mm
Other:
- outline, holes or cut-outs redrawn
- board text added: "PhoZL 2.0.2"
- board text added: "ZL"
- board text added: "ZR"
- board text added: "github.com/sean44104/PhoZL"
- board text removed: "PhobGCC 2.0.2"
- board text removed: "github.com/PhobGCC"
